Commit message: Modified code structure and Simulation

File: Virtual_model/Qube_Servo_3.urdf (robot description, URDF)
Before this commit: robot qube_servo_3, 2 links, 1 joints
Links:
- removed link rotor
- added link arm_link, mass 0.095; collision box size=0.085 0.010 0.006; visual box size=0.085 0.010 0.006
- added link pendulum_link, mass 0.024; collision cylinder length=0.129 radius=0.006; visual cylinder length=0.129 radius=0.006
- added link world
- link base_link: geometry collision box size=0.090 0.090 0.090; visual box size=0.090 0.090 0.090
Joints:
- added joint pendulum_joint: type continuous, parent arm_link, child pendulum_link, origin xyz=0.085 0 0 rpy=0 0 0, axis 1 0 0, limit effort=0.0 velocity=100.0
- added joint world_to_base: type fixed, parent world, child base_link, origin xyz=0 0 0 rpy=0 0 0
- joint motor_joint: child rotor -> arm_link; limit effort=18.0 velocity=100.0 -> lower=1.5708 upper=4.7124 effort=18.0 velocity=100.0; origin xyz=0 0 0.075 rpy=0 0 0 -> xyz=0 0 0.090 rpy=0 0 0; type continuous -> revolute
